Commit message: update urdf file
create a correct urdf file to display model correctly

Signed-off-by: mxlfrbt <mxlfrbt@icloud.com>

File: ros/src/mikrik_description/urdf/mikrik.xacro (robot description, xacro)
@@ -4,5 +4,5 @@
 	xmlns:xacro="http://www.ros.org/wiki/xacro">
 	<xacro:property name="clearance" value="0.018" />
-	<xacro:property name="wheel_radius" value="0.03195"/>
+	<xacro:property name="wheel_radius" value="0.0325"/>
 	<xacro:property name="wheel_separation" value="0.128"/>
 	<xacro:property name="wheel_width" value="0.026"/>

File: ros/src/mikrik_description/urdf/mikrik_left_wheel.xacro (robot description, xacro)
@@ -3,20 +3,4 @@
 <robot name="mikrik"
 	xmlns:xacro="http://www.ros.org/wiki/xacro">
-	<!-- left_wheel -->
-	<link name="mikrik_left_wheel">
-		<visual>
-			<origin xyz="0 0 0" rpy="0 0 0" />
-			<geometry>
-				<cylinder length="0.026" radius="0.0325"/>
-			</geometry>
-			<material name="Green" />
-		</visual>
-		<collision>
-			<origin xyz="0 0 0" rpy="0 0 0" />
-			<geometry>
-				<cylinder length="0.026" radius="0.0325"/>
-			</geometry>
-		</collision>
-	</link>
 	<!-- left_wheel_geometry -->
 	<link name="left_wheel">
@@ -35,9 +19,4 @@
 		</collision>
 	</link>
-	<joint name="left_wheel_to_mikrik_left_wheel" type="fixed">
-		<origin xyz="0 0 0" rpy="0 0 0" />
-		<parent link="left_wheel" />
-		<child link="mikrik_left_wheel" />
-	</joint>
 	<joint name="left_wheel_to_base" type="continuous">
 		<origin xyz="0 0.068 0.0145" rpy="0 0 0" />

File: ros/src/mikrik_description/urdf/mikrik_right_wheel.xacro (robot description, xacro)
@@ -3,20 +3,4 @@
 <robot name="mikrik"
 	xmlns:xacro="http://www.ros.org/wiki/xacro">
-	<!-- right_wheel -->
-	<link name="mikrik_right_wheel">
-		<visual>
-			<origin xyz="0 0 0" rpy="0 0 0" />
-			<geometry>
-				<cylinder length="0.026" radius="0.0325"/>
-			</geometry>
-			<material name="Green" />
-		</visual>
-		<collision>
-			<origin xyz="0 0 0" rpy="0 0 0" />
-			<geometry>
-				<cylinder length="0.026" radius="0.0325"/>
-			</geometry>
-		</collision>
-	</link>
 	<!-- right_wheel_geometry -->
 	<link name="right_wheel">
@@ -35,9 +19,4 @@
 		</collision>
 	</link>
-	<joint name="right_wheel_to_mikrik_right_wheel" type="fixed">
-		<origin xyz="0 0 0" rpy="0 0 0" />
-		<parent link="right_wheel" />
-		<child link="mikrik_right_wheel" />
-	</joint>
 	<joint name="right_wheel_to_base" type="continuous">
 		<origin xyz="0 -0.068 0.0145" rpy="0 0 0" />
